Commit message: Rviz visualization works! Credit to @janieleung

File: resources/go1/urdf/depthCamera.xacro (robot description, xacro)
@@ -17,5 +17,5 @@
             <origin xyz="0 0 0" rpy="0 0 0"/>
             <geometry>
-                <mesh filename="../meshes/depthCamera.dae" scale="1 1 1"/>
+                <mesh filename="package://galileo_go1_description/meshes/depthCamera.dae" scale="1 1 1"/>
             </geometry>
             </visual>

File: resources/go1/urdf/go1.urdf (robot description, URDF)
Before this commit: robot go1, 47 links, 46 joints
Links:
- link FL_calf: geometry collision box size=0.213 0.016 0.016; visual mesh filename=package://galileo_go1_description/meshes/calf.dae scale=1 1 1
- link FL_hip: geometry collision cylinder length=0.04 radius=0.046; visual mesh filename=package://galileo_go1_description/meshes/hip.dae scale=1 1 1
- link FL_thigh: geometry collision box size=0.213 0.0245 0.034; visual mesh filename=package://galileo_go1_description/meshes/thigh.dae scale=1 1 1
- link FR_calf: geometry collision box size=0.213 0.016 0.016; visual mesh filename=package://galileo_go1_description/meshes/calf.dae scale=1 1 1
- link FR_hip: geometry collision cylinder length=0.04 radius=0.046; visual mesh filename=package://galileo_go1_description/meshes/hip.dae scale=1 1 1
- link FR_thigh: geometry collision box size=0.213 0.0245 0.034; visual mesh filename=package://galileo_go1_description/meshes/thigh_mirror.dae scale=1 1 1
- link RL_calf: geometry collision box size=0.213 0.016 0.016; visual mesh filename=package://galileo_go1_description/meshes/calf.dae scale=1 1 1
- link RL_hip: geometry collision cylinder length=0.04 radius=0.046; visual mesh filename=package://galileo_go1_description/meshes/hip.dae scale=1 1 1
- link RL_thigh: geometry collision box size=0.213 0.0245 0.034; visual mesh filename=package://galileo_go1_description/meshes/thigh.dae scale=1 1 1
- link RR_calf: geometry collision box size=0.213 0.016 0.016; visual mesh filename=package://galileo_go1_description/meshes/calf.dae scale=1 1 1
- link RR_hip: geometry collision cylinder length=0.04 radius=0.046; visual mesh filename=package://galileo_go1_description/meshes/hip.dae scale=1 1 1
- link RR_thigh: geometry collision box size=0.213 0.0245 0.034; visual mesh filename=package://galileo_go1_description/meshes/thigh_mirror.dae scale=1 1 1
- link camera_chin: geometry collision box size=.001 .001 .001; visual mesh filename=package://galileo_go1_description/meshes/depthCamera.dae scale=1 1 1
- link camera_face: geometry collision box size=.001 .001 .001; visual mesh filename=package://galileo_go1_description/meshes/depthCamera.dae scale=1 1 1
- link camera_left: geometry collision box size=.001 .001 .001; visual mesh filename=package://galileo_go1_description/meshes/depthCamera.dae scale=1 1 1
- link camera_rearDown: geometry collision box size=.001 .001 .001; visual mesh filename=package://galileo_go1_description/meshes/depthCamera.dae scale=1 1 1
- link camera_right: geometry collision box size=.001 .001 .001; visual mesh filename=package://galileo_go1_description/meshes/depthCamera.dae scale=1 1 1
- link trunk: geometry collision box size=0.3762 0.0935 0.114; visual mesh filename=package://galileo_go1_description/meshes/trunk.dae scale=1 1 1
- link ultraSound_face: geometry collision box size=.001 .001 .001; visual mesh filename=package://galileo_go1_description/meshes/ultraSound.dae scale=1 1 1
- link ultraSound_left: geometry collision box size=.001 .001 .001; visual mesh filename=package://galileo_go1_description/meshes/ultraSound.dae scale=1 1 1
- link ultraSound_right: geometry collision box size=.001 .001 .001; visual mesh filename=package://galileo_go1_description/meshes/ultraSound.dae scale=1 1 1

File: resources/go1/urdf/leg.xacro (robot description, xacro)
@@ -58,5 +58,5 @@
                 </xacro:if>
                 <geometry>
-                    <mesh filename="../meshes/hip.dae" scale="1 1 1"/>
+                    <mesh filename="package://galileo_go1_description/meshes/hip.dae" scale="1 1 1"/>
                 </geometry>
                 <!-- <material name="orange"/> -->
@@ -118,8 +118,8 @@
                 <geometry>
                     <xacro:if value="${mirror_dae == True}">
-                        <mesh filename="../meshes/thigh.dae" scale="1 1 1"/>
+                        <mesh filename="package://galileo_go1_description/meshes/thigh.dae" scale="1 1 1"/>
                     </xacro:if>
                     <xacro:if value="${mirror_dae == False}">
-                        <mesh filename="../meshes/thigh_mirror.dae" scale="1 1 1"/>
+                        <mesh filename="package://galileo_go1_description/meshes/thigh_mirror.dae" scale="1 1 1"/>
                     </xacro:if>
                 </geometry>
@@ -181,5 +181,5 @@
                 <origin rpy="0 0 0" xyz="0 0 0"/>
                 <geometry>
-                    <mesh filename="../meshes/calf.dae" scale="1 1 1"/>
+                    <mesh filename="package://galileo_go1_description/meshes/calf.dae" scale="1 1 1"/>
                 </geometry>
                 <!-- <material name="orange"/> -->

File: resources/go1/urdf/robot.xacro (robot description, xacro)
@@ -37,5 +37,5 @@
             <origin rpy="0 0 0" xyz="0 0 0"/>
             <geometry>
-                <mesh filename="../meshes/trunk.dae" scale="1 1 1"/>
+                <mesh filename="package://galileo_go1_description/meshes/trunk.dae" scale="1 1 1"/>
             </geometry>
             <!-- <material name="orange"/> -->

File: resources/go1/urdf/ultraSound.xacro (robot description, xacro)
@@ -17,5 +17,5 @@
             <origin xyz="0 0 0" rpy="0 0 0"/>
             <geometry>
-                <mesh filename="../meshes/ultraSound.dae" scale="1 1 1"/>
+                <mesh filename="package://galileo_go1_description/meshes/ultraSound.dae" scale="1 1 1"/>
             </geometry>
             <material name="black"/>
