Commit message: Issue #45

File: resources/go1/urdf/go1.urdf (robot description, URDF)
Before this commit: robot go1, 47 links, 46 joints
Joints:
- joint world_fixed: type floating -> fixed

File: resources/go1/urdf/robot.xacro (robot description, xacro)
@@ -15,5 +15,5 @@
     <!-- Debug mode will hung up the robot, use "true" or "false" to switch it. -->
     <link name="world"/>
-    <joint name="world_fixed" type="floating">
+    <joint name="world_fixed" type="fixed">
         <origin xyz="0 0 0" rpy="0 0 0"/>
         <parent link="world"/>

File: resources/huron/urdf/huron.urdf (robot description, URDF)
Before this commit: robot huron, 27 links, 26 joints
Links:
- removed link base_link
- added link base
- added link world
- link base_footprint: geometry collision mesh filename=resources/huron/meshes/base_link.STL scale=1 1 1; visual mesh filename=resources/huron/meshes/base_link.STL scale=1 1 1
- link l1_foot_ft_link: geometry visual mesh filename=resources/huron/meshes/l1_foot_ft_link.STL scale=1 1 1
- link l2_foot_ft_link: geometry visual mesh filename=resources/huron/meshes/l2_foot_ft_link.STL scale=1 1 1
- link l3_foot_ft_link: geometry visual mesh filename=resources/huron/meshes/l3_foot_ft_link.STL scale=1 1 1
- link l4_foot_ft_link: geometry visual mesh filename=resources/huron/meshes/l4_foot_ft_link.STL scale=1 1 1
- link l_ankle_pitch_link: geometry collision mesh filename=resources/huron/meshes/l_ankle_pitch_link.STL scale=1 1 1; visual mesh filename=resources/huron/meshes/l_ankle_pitch_link.STL scale=1 1 1
- link l_ankle_roll_link: geometry collision mesh filename=resources/huron/meshes/l_ankle_roll_link.STL scale=1 1 1; visual mesh filename=resources/huron/meshes/l_ankle_roll_link.STL scale=1 1 1
- link l_hip_pitch_link: geometry collision mesh filename=resources/huron/meshes/l_hip_pitch_link.STL scale=1 1 1; visual mesh filename=resources/huron/meshes/l_hip_pitch_link.STL scale=1 1 1
- link l_hip_roll_link: geometry collision mesh filename=resources/huron/meshes/l_hip_roll_link.STL scale=1 1 1; visual mesh filename=resources/huron/meshes/l_hip_roll_link.STL scale=1 1 1
- link l_hip_yaw_link: geometry collision mesh filename=resources/huron/meshes/l_hip_yaw_link.STL scale=1 1 1; visual mesh filename=resources/huron/meshes/l_hip_yaw_link.STL scale=1 1 1
- link l_knee_pitch_link: geometry collision mesh filename=resources/huron/meshes/l_knee_pitch_link.STL scale=1 1 1; visual mesh filename=resources/huron/meshes/l_knee_pitch_link.STL scale=1 1 1
- link r1_foot_ft_link: geometry visual mesh filename=resources/huron/meshes/r1_foot_ft_link.STL scale=1 1 1
- link r2_foot_ft_link: geometry visual mesh filename=resources/huron/meshes/r2_foot_ft_link.STL scale=1 1 1
- link r3_foot_ft_link: geometry visual mesh filename=resources/huron/meshes/r3_foot_ft_link.STL scale=1 1 1
- link r4_foot_ft_link: geometry visual mesh filename=resources/huron/meshes/r4_foot_ft_link.STL scale=1 1 1
- link r_ankle_pitch_link: geometry collision mesh filename=resources/huron/meshes/r_ankle_pitch_link.STL scale=1 1 1; visual mesh filename=resources/huron/meshes/r_ankle_pitch_link.STL scale=1 1 1
- link r_ankle_roll_link: geometry collision mesh filename=resources/huron/meshes/r_ankle_roll_link.STL scale=1 1 1; visual mesh filename=resources/huron/meshes/r_ankle_roll_link.STL scale=1 1 1
- link r_hip_pitch_link: geometry collision mesh filename=resources/huron/meshes/r_hip_pitch_link.STL scale=1 1 1; visual mesh filename=resources/huron/meshes/r_hip_pitch_link.STL scale=1 1 1
- link r_hip_roll_link: geometry collision mesh filename=resources/huron/meshes/r_hip_roll_link.STL scale=1 1 1; visual mesh filename=resources/huron/meshes/r_hip_roll_link.STL scale=1 1 1
- link r_hip_yaw_link: geometry collision mesh filename=resources/huron/meshes/r_hip_yaw_link.STL scale=1 1 1; visual mesh filename=resources/huron/meshes/r_hip_yaw_link.STL scale=1 1 1
- link r_knee_pitch_link: geometry collision mesh filename=resources/huron/meshes/r_knee_pitch_link.STL scale=1 1 1; visual mesh filename=resources/huron/meshes/r_knee_pitch_link.STL scale=1 1 1
Joints:
- added joint world_fixed: type fixed, parent world, child base, origin xyz=0 0 0 rpy=0 0 0
- joint base_fixed: parent base_link -> base

File: resources/huron/urdf/huron.xacro (robot description, xacro)
@@ -18,8 +18,16 @@
         <child link="base_link"/>
     </joint> -->
-    <link name="base_link"></link>
+    <link name="world"></link>
+    <!-- floating link -->
+    <!-- <xacro:huron_floating parent="world" child="base"/> -->
+    <joint name="world_fixed" type="fixed">
+        <origin xyz="0 0 0" rpy="0 0 0"/>
+        <parent link="world"/>
+        <child link="base"/>
+    </joint>
+    <link name="base"></link>
     <joint name="base_fixed" type="fixed">
         <origin xyz="0 0 0" rpy="0 0 0"/>
-        <parent link="base_link"/>
+        <parent link="base"/>
         <child link="base_footprint"/>
     </joint>

Commit message: Got Go1 to walk in rviz!

File: resources/go1/urdf/go1.urdf (robot description, URDF)
Before this commit: robot go1, 47 links, 46 joints
Links:
- link FL_calf: geometry collision box size=0.213 0.016 0.016; visual mesh filename=package://galileo_go1_description/meshes/calf.dae scale=1 1 1
- link FL_hip: geometry collision cylinder length=0.04 radius=0.046; visual mesh filename=package://galileo_go1_description/meshes/hip.dae scale=1 1 1
- link FL_thigh: geometry collision box size=0.213 0.0245 0.034; visual mesh filename=package://galileo_go1_description/meshes/thigh.dae scale=1 1 1
- link FR_calf: geometry collision box size=0.213 0.016 0.016; visual mesh filename=package://galileo_go1_description/meshes/calf.dae scale=1 1 1
- link FR_hip: geometry collision cylinder length=0.04 radius=0.046; visual mesh filename=package://galileo_go1_description/meshes/hip.dae scale=1 1 1
- link FR_thigh: geometry collision box size=0.213 0.0245 0.034; visual mesh filename=package://galileo_go1_description/meshes/thigh_mirror.dae scale=1 1 1
- link RL_calf: geometry collision box size=0.213 0.016 0.016; visual mesh filename=package://galileo_go1_description/meshes/calf.dae scale=1 1 1
- link RL_hip: geometry collision cylinder length=0.04 radius=0.046; visual mesh filename=package://galileo_go1_description/meshes/hip.dae scale=1 1 1
- link RL_thigh: geometry collision box size=0.213 0.0245 0.034; visual mesh filename=package://galileo_go1_description/meshes/thigh.dae scale=1 1 1
- link RR_calf: geometry collision box size=0.213 0.016 0.016; visual mesh filename=package://galileo_go1_description/meshes/calf.dae scale=1 1 1
- link RR_hip: geometry collision cylinder length=0.04 radius=0.046; visual mesh filename=package://galileo_go1_description/meshes/hip.dae scale=1 1 1
- link RR_thigh: geometry collision box size=0.213 0.0245 0.034; visual mesh filename=package://galileo_go1_description/meshes/thigh_mirror.dae scale=1 1 1
- link camera_chin: geometry collision box size=.001 .001 .001; visual mesh filename=package://galileo_go1_description/meshes/depthCamera.dae scale=1 1 1
- link camera_face: geometry collision box size=.001 .001 .001; visual mesh filename=package://galileo_go1_description/meshes/depthCamera.dae scale=1 1 1
- link camera_left: geometry collision box size=.001 .001 .001; visual mesh filename=package://galileo_go1_description/meshes/depthCamera.dae scale=1 1 1
- link camera_rearDown: geometry collision box size=.001 .001 .001; visual mesh filename=package://galileo_go1_description/meshes/depthCamera.dae scale=1 1 1
- link camera_right: geometry collision box size=.001 .001 .001; visual mesh filename=package://galileo_go1_description/meshes/depthCamera.dae scale=1 1 1
- link trunk: geometry collision box size=0.3762 0.0935 0.114; visual mesh filename=package://galileo_go1_description/meshes/trunk.dae scale=1 1 1
- link ultraSound_face: geometry collision box size=.001 .001 .001; visual mesh filename=package://galileo_go1_description/meshes/ultraSound.dae scale=1 1 1
- link ultraSound_left: geometry collision box size=.001 .001 .001; visual mesh filename=package://galileo_go1_description/meshes/ultraSound.dae scale=1 1 1
- link ultraSound_right: geometry collision box size=.001 .001 .001; visual mesh filename=package://galileo_go1_description/meshes/ultraSound.dae scale=1 1 1

Commit message: Galileo solves trotting in 15ms per iterationgit statusgit status

File: resources/go1/urdf/go1.urdf (robot description, URDF)
Before this commit: robot go1, 47 links, 46 joints
Links:
- removed link FL_calf
- removed link FL_calf_rotor
- removed link FL_foot
- removed link FL_hip
- removed link FL_hip_rotor
- removed link FL_thigh
- removed link FL_thigh_rotor
- removed link FR_calf
- removed link FR_calf_rotor
- removed link FR_foot
- removed link FR_hip
- removed link FR_hip_rotor
- removed link FR_thigh
- removed link FR_thigh_rotor
- removed link RL_calf
- removed link RL_calf_rotor
- removed link RL_foot
- removed link RL_hip
- removed link RL_hip_rotor
- removed link RL_thigh
- removed link RL_thigh_rotor
- removed link RR_calf
- removed link RR_calf_rotor
- removed link RR_foot
- removed link RR_hip
- removed link RR_hip_rotor
- removed link RR_thigh
- removed link RR_thigh_rotor
- removed link camera_chin
- removed link camera_face
- removed link camera_laserscan_link_left
- removed link camera_laserscan_link_right
- removed link camera_left
- removed link camera_optical_chin
- removed link camera_optical_face
- removed link camera_optical_left
- removed link camera_optical_rearDown
- removed link camera_optical_right
- removed link camera_rearDown
- removed link camera_right
- removed link imu_link
- removed link trunk
- removed link ultraSound_face
- removed link ultraSound_left
- removed link ultraSound_right
- removed link world
- added link LF_FOOT, mass 0.06; collision sphere radius=0.02; visual sphere radius=0.01
- added link LF_calf, mass 0.135862; collision box size=0.213 0.016 0.016; visual mesh filename=package://galileo_go1_description/meshes/calf.dae scale=1 1 1
- added link LF_hip, mass 0.591; collision cylinder length=0.04 radius=0.046; visual mesh filename=package://galileo_go1_description/meshes/hip.dae scale=1 1 1
- added link LF_thigh, mass 0.92; collision box size=0.213 0.0245 0.034; collision cylinder length=0.032 radius=0.041
- added link LH_FOOT, mass 0.06; collision sphere radius=0.02; visual sphere radius=0.01
- added link LH_calf, mass 0.135862; collision box size=0.213 0.016 0.016; visual mesh filename=package://galileo_go1_description/meshes/calf.dae scale=1 1 1
- added link LH_hip, mass 0.591; collision cylinder length=0.04 radius=0.046; visual mesh filename=package://galileo_go1_description/meshes/hip.dae scale=1 1 1
- added link LH_thigh, mass 0.92; collision box size=0.213 0.0245 0.034; collision cylinder length=0.032 radius=0.041
- added link RF_FOOT, mass 0.06; collision sphere radius=0.02; visual sphere radius=0.01
- added link RF_calf, mass 0.135862; collision box size=0.213 0.016 0.016; visual mesh filename=package://galileo_go1_description/meshes/calf.dae scale=1 1 1
- added link RF_hip, mass 0.591; collision cylinder length=0.04 radius=0.046; visual mesh filename=package://galileo_go1_description/meshes/hip.dae scale=1 1 1
- added link RF_thigh, mass 0.92; collision box size=0.213 0.0245 0.034; collision cylinder length=0.032 radius=0.041
- added link RH_FOOT, mass 0.06; collision sphere radius=0.02; visual sphere radius=0.01
- added link RH_calf, mass 0.135862; collision box size=0.213 0.016 0.016; visual mesh filename=package://galileo_go1_description/meshes/calf.dae scale=1 1 1
- added link RH_hip, mass 0.591; collision cylinder length=0.04 radius=0.046; visual mesh filename=package://galileo_go1_description/meshes/hip.dae scale=1 1 1
- added link RH_thigh, mass 0.92; collision box size=0.213 0.0245 0.034; collision cylinder length=0.032 radius=0.041
- added link unitree_imu, mass 0.01; visual box size=0.015 0.015 0.004
- link base: mass None -> 5.204; geometry collision box size=0.3762 0.0935 0.114; visual mesh filename=package://galileo_go1_description/meshes/trunk.dae scale=1 1 1
Joints:
- removed joint FL_calf_joint
- removed joint FL_calf_rotor_joint
- removed joint FL_foot_fixed
- removed joint FL_hip_joint
- removed joint FL_hip_rotor_joint
- removed joint FL_thigh_joint
- removed joint FL_thigh_rotor_joint
- removed joint FR_calf_joint
- removed joint FR_calf_rotor_joint
- removed joint FR_foot_fixed
- removed joint FR_hip_joint
- removed joint FR_hip_rotor_joint
- removed joint FR_thigh_joint
- removed joint FR_thigh_rotor_joint
- removed joint RL_calf_joint
- removed joint RL_calf_rotor_joint
- removed joint RL_foot_fixed
- removed joint RL_hip_joint
- removed joint RL_hip_rotor_joint
- removed joint RL_thigh_joint
- removed joint RL_thigh_rotor_joint
- removed joint RR_calf_joint
- removed joint RR_calf_rotor_joint
- removed joint RR_foot_fixed
- removed joint RR_hip_joint
- removed joint RR_hip_rotor_joint
- removed joint RR_thigh_joint
- removed joint RR_thigh_rotor_joint
- removed joint camera_joint_chin
- removed joint camera_joint_face
- removed joint camera_joint_left
- removed joint camera_joint_rearDown
- removed joint camera_joint_right
- removed joint camera_laserscan_joint_left
- removed joint camera_laserscan_joint_right
- removed joint camera_optical_joint_chin
- removed joint camera_optical_joint_face
- removed joint camera_optical_joint_left
- removed joint camera_optical_joint_rearDown
- removed joint camera_optical_joint_right
- removed joint floating_base
- removed joint imu_joint
- removed joint ultraSound_joint_face
- removed joint ultraSound_joint_left
- removed joint ultraSound_joint_right
- removed joint world_fixed
- added joint LF_HAA: type revolute, parent base, child LF_hip, origin xyz=0.1881 0.04675 0 rpy=0 0 0, axis 1 0 0, limit lower=-0.863 upper=0.863 effort=23.7 velocity=30.1
- added joint LF_HFE: type revolute, parent LF_hip, child LF_thigh, origin xyz=0 0.08 0 rpy=0 0 0, axis 0 1 0, limit lower=-0.686 upper=4.501 effort=23.7 velocity=30.1
- added joint LF_KFE: type revolute, parent LF_thigh, child LF_calf, origin xyz=0 0 -0.213 rpy=0 0 0, axis 0 1 0, limit lower=-2.818 upper=-0.888 effort=35.55 velocity=20.06
- added joint LF_foot_fixed: type fixed, parent LF_calf, child LF_FOOT, origin xyz=0 0 -0.213 rpy=0 0 0
- added joint LH_HAA: type revolute, parent base, child LH_hip, origin xyz=-0.1881 0.04675 0 rpy=0 0 0, axis 1 0 0, limit lower=-0.863 upper=0.863 effort=23.7 velocity=30.1
- added joint LH_HFE: type revolute, parent LH_hip, child LH_thigh, origin xyz=0 0.08 0 rpy=0 0 0, axis 0 1 0, limit lower=-0.686 upper=4.501 effort=23.7 velocity=30.1
- added joint LH_KFE: type revolute, parent LH_thigh, child LH_calf, origin xyz=0 0 -0.213 rpy=0 0 0, axis 0 1 0, limit lower=-2.818 upper=-0.888 effort=35.55 velocity=20.06
- added joint LH_foot_fixed: type fixed, parent LH_calf, child LH_FOOT, origin xyz=0 0 -0.213 rpy=0 0 0
- added joint RF_HAA: type revolute, parent base, child RF_hip, origin xyz=0.1881 -0.04675 0 rpy=0 0 0, axis 1 0 0, limit lower=-0.863 upper=0.863 effort=23.7 velocity=30.1
- added joint RF_HFE: type revolute, parent RF_hip, child RF_thigh, origin xyz=0 -0.08 0 rpy=0 0 0, axis 0 1 0, limit lower=-0.686 upper=4.501 effort=23.7 velocity=30.1
- added joint RF_KFE: type revolute, parent RF_thigh, child RF_calf, origin xyz=0 0 -0.213 rpy=0 0 0, axis 0 1 0, limit lower=-2.818 upper=-0.888 effort=35.55 velocity=20.06
- added joint RF_foot_fixed: type fixed, parent RF_calf, child RF_FOOT, origin xyz=0 0 -0.213 rpy=0 0 0
- added joint RH_HAA: type revolute, parent base, child RH_hip, origin xyz=-0.1881 -0.04675 0 rpy=0 0 0, axis 1 0 0, limit lower=-0.863 upper=0.863 effort=23.7 velocity=30.1
- added joint RH_HFE: type revolute, parent RH_hip, child RH_thigh, origin xyz=0 -0.08 0 rpy=0 0 0, axis 0 1 0, limit lower=-0.686 upper=4.501 effort=23.7 velocity=30.1
- added joint RH_KFE: type revolute, parent RH_thigh, child RH_calf, origin xyz=0 0 -0.213 rpy=0 0 0, axis 0 1 0, limit lower=-2.818 upper=-0.888 effort=35.55 velocity=20.06
- added joint RH_foot_fixed: type fixed, parent RH_calf, child RH_FOOT, origin xyz=0 0 -0.213 rpy=0 0 0
- added joint unitree_imu_joint: type fixed, parent base, child unitree_imu, origin xyz=0. 0. 0. rpy=0. 0. 0.
