Commit message: HURON Ros launch

File: resources/huron/urdf/huron.urdf (robot description, URDF)
Before this commit: robot huron, 28 links, 27 joints
Links:
- link base_footprint: geometry collision mesh filename=package://galileo_huron_description/meshes/base_link.STL scale=1 1 1; visual mesh filename=package://galileo_huron_description/meshes/base_link.STL scale=1 1 1
- link l1_foot_ft_link: geometry visual mesh filename=package://galileo_huron_description/meshes/l1_foot_ft_link.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 scale=1 1 1
- link l2_foot_ft_link: geometry visual mesh filename=package://galileo_huron_description/meshes/l2_foot_ft_link.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 scale=1 1 1
- link l3_foot_ft_link: geometry visual mesh filename=package://galileo_huron_description/meshes/l3_foot_ft_link.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 scale=1 1 1
- link l4_foot_ft_link: geometry visual mesh filename=package://galileo_huron_description/meshes/l4_foot_ft_link.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 scale=1 1 1
- link l_ankle_pitch_link: geometry collision mesh filename=package://galileo_huron_description/meshes/l_ankle_pitch_li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 scale=1 1 1; visual mesh filename=package://galileo_huron_description/meshes/l_ankle_pitch_li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 scale=1 1 1
- link l_ankle_roll_link: geometry collision mesh filename=package://galileo_huron_description/meshes/l_ankle_roll_lin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 scale=1 1 1; visual mesh filename=package://galileo_huron_description/meshes/l_ankle_roll_lin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 scale=1 1 1
- link l_hip_pitch_link: geometry collision mesh filename=package://galileo_huron_description/meshes/l_hip_pitch_link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 scale=1 1 1; visual mesh filename=package://galileo_huron_description/meshes/l_hip_pitch_link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 scale=1 1 1
- link l_hip_roll_link: geometry collision mesh filename=package://galileo_huron_description/meshes/l_hip_roll_link.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 scale=1 1 1; visual mesh filename=package://galileo_huron_description/meshes/l_hip_roll_link.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 scale=1 1 1
- link l_hip_yaw_link: geometry collision mesh filename=package://galileo_huron_description/meshes/l_hip_yaw_link.S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 scale=1 1 1; visual mesh filename=package://galileo_huron_description/meshes/l_hip_yaw_link.S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 scale=1 1 1
- link l_knee_pitch_link: geometry collision mesh filename=package://galileo_huron_description/meshes/l_knee_pitch_lin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 scale=1 1 1; visual mesh filename=package://galileo_huron_description/meshes/l_knee_pitch_lin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 scale=1 1 1
- link r1_foot_ft_link: geometry visual mesh filename=package://galileo_huron_description/meshes/r1_foot_ft_link.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 scale=1 1 1
- link r2_foot_ft_link: geometry visual mesh filename=package://galileo_huron_description/meshes/r2_foot_ft_link.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 scale=1 1 1
- link r3_foot_ft_link: geometry visual mesh filename=package://galileo_huron_description/meshes/r3_foot_ft_link.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 scale=1 1 1
- link r4_foot_ft_link: geometry visual mesh filename=package://galileo_huron_description/meshes/r4_foot_ft_link.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 scale=1 1 1
- link r_ankle_pitch_link: geometry collision mesh filename=package://galileo_huron_description/meshes/r_ankle_pitch_li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 scale=1 1 1; visual mesh filename=package://galileo_huron_description/meshes/r_ankle_pitch_li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 scale=1 1 1
- link r_ankle_roll_link: geometry collision mesh filename=package://galileo_huron_description/meshes/r_ankle_roll_lin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 scale=1 1 1; visual mesh filename=package://galileo_huron_description/meshes/r_ankle_roll_lin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 scale=1 1 1
- link r_hip_pitch_link: geometry collision mesh filename=package://galileo_huron_description/meshes/r_hip_pitch_link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 scale=1 1 1; visual mesh filename=package://galileo_huron_description/meshes/r_hip_pitch_link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 scale=1 1 1
- link r_hip_roll_link: geometry collision mesh filename=package://galileo_huron_description/meshes/r_hip_roll_link.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 scale=1 1 1; visual mesh filename=package://galileo_huron_description/meshes/r_hip_roll_link.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 scale=1 1 1
- link r_hip_yaw_link: geometry collision mesh filename=package://galileo_huron_description/meshes/r_hip_yaw_link.S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 scale=1 1 1; visual mesh filename=package://galileo_huron_description/meshes/r_hip_yaw_link.S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 scale=1 1 1
- link r_knee_pitch_link: geometry collision mesh filename=package://galileo_huron_description/meshes/r_knee_pitch_lin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 scale=1 1 1; visual mesh filename=package://galileo_huron_description/meshes/r_knee_pitch_lin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 scale=1 1 1

File: resources/huron/urdf/huron_visuals.xacro (robot description, xacro)
@@ -6,5 +6,5 @@
         <origin xyz="0 0 0" rpy="0 0 0" />
         <geometry>
-            <mesh filename="package://huron_description/meshes/base_link.STL" scale="1 1 1" />
+            <mesh filename="package://galileo_huron_description/meshes/base_link.STL" scale="1 1 1" />
         </geometry>
         <material name="grey"/>
@@ -30,5 +30,5 @@
         <origin xyz="0 0 0" rpy="0 0 0" />
         <geometry>
-            <mesh filename="package://huron_description/meshes/l_hip_yaw_link.STL" scale="1 1 1" />
+            <mesh filename="package://galileo_huron_description/meshes/l_hip_yaw_link.STL" scale="1 1 1" />
         </geometry>
         <material name="grey"/>
@@ -38,5 +38,5 @@
         <origin xyz="0 0 0" rpy="0 0 0" />
         <geometry>
-            <mesh filename="package://huron_description/meshes/l_hip_roll_link.STL" scale="1 1 1" />
+            <mesh filename="package://galileo_huron_description/meshes/l_hip_roll_link.STL" scale="1 1 1" />
         </geometry>
         <material name="grey"/>
@@ -46,5 +46,5 @@
         <origin xyz="0 0 0" rpy="0 0 0" />
         <geometry>
-            <mesh filename="package://huron_description/meshes/l_hip_pitch_link.STL" scale="1 1 1" />
+            <mesh filename="package://galileo_huron_description/meshes/l_hip_pitch_link.STL" scale="1 1 1" />
         </geometry>
         <material name="grey"/>
@@ -54,5 +54,5 @@
         <origin xyz="0 0 0" rpy="0 0 0" />
         <geometry>
-            <mesh filename="package://huron_description/meshes/l_knee_pitch_link.STL" scale="1 1 1" />
+            <mesh filename="package://galileo_huron_description/meshes/l_knee_pitch_link.STL" scale="1 1 1" />
         </geometry>
         <material name="grey"/>
@@ -62,5 +62,5 @@
         <origin xyz="0 0 0" rpy="0 0 0" />
         <geometry>
-            <mesh filename="package://huron_description/meshes/l_ankle_pitch_link.STL" scale="1 1 1" />
+            <mesh filename="package://galileo_huron_description/meshes/l_ankle_pitch_link.STL" scale="1 1 1" />
         </geometry>
         <material name="">
@@ -72,5 +72,5 @@
         <origin xyz="0 0 0" rpy="0 0 0" />
         <geometry>
-            <mesh filename="package://huron_description/meshes/l_ankle_roll_link.STL" scale="1 1 1" />
+            <mesh filename="package://galileo_huron_description/meshes/l_ankle_roll_link.STL" scale="1 1 1" />
         </geometry>
         <material name="">
@@ -82,5 +82,5 @@
         <origin xyz="0 0 0" rpy=" 0 0 0" />
         <geometry>
-            <mesh filename="package://huron_description/meshes/l1_foot_ft_link.STL" scale="1 1 1" />
+            <mesh filename="package://galileo_huron_description/meshes/l1_foot_ft_link.STL" scale="1 1 1" />
         </geometry>
         <material name="green"/>
@@ -90,5 +90,5 @@
         <origin xyz="0 0 0" rpy=" 0 0 0" />
         <geometry>
-            <mesh filename="package://huron_description/meshes/l2_foot_ft_link.STL" scale="1 1 1" />
+            <mesh filename="package://galileo_huron_description/meshes/l2_foot_ft_link.STL" scale="1 1 1" />
         </geometry>
         <material name="green"/>
@@ -98,5 +98,5 @@
         <origin xyz="0 0 0" rpy=" 0 0 0" />
         <geometry>
-            <mesh filename="package://huron_description/meshes/l3_foot_ft_link.STL" scale="1 1 1" />
+            <mesh filename="package://galileo_huron_description/meshes/l3_foot_ft_link.STL" scale="1 1 1" />
         </geometry>
         <material name="green"/>
@@ -106,5 +106,5 @@
         <origin xyz="0 0 0" rpy=" 0 0 0" />
         <geometry>
-            <mesh filename="package://huron_description/meshes/l4_foot_ft_link.STL" scale="1 1 1" />
+            <mesh filename="package://galileo_huron_description/meshes/l4_foot_ft_link.STL" scale="1 1 1" />
         </geometry>
         <material name="green"/>
@@ -114,5 +114,5 @@
         <origin xyz="0 0 0" rpy="0 0 0" />
         <geometry>
-            <mesh filename="package://huron_description/meshes/r_hip_yaw_link.STL" scale="1 1 1" />
+            <mesh filename="package://galileo_huron_description/meshes/r_hip_yaw_link.STL" scale="1 1 1" />
         </geometry>
         <material name="grey"/>
@@ -122,5 +122,5 @@
         <origin xyz="0 0 0" rpy="0 0 0" />
         <geometry>
-            <mesh filename="package://huron_description/meshes/r_hip_roll_link.STL" scale="1 1 1" />
+            <mesh filename="package://galileo_huron_description/meshes/r_hip_roll_link.STL" scale="1 1 1" />
         </geometry>
         <material name="grey"/>
@@ -130,5 +130,5 @@
         <origin xyz="0 0 0" rpy="0 0 0" />
         <geometry>
-            <mesh filename="package://huron_description/meshes/r_hip_pitch_link.STL" scale="1 1 1" />
+            <mesh filename="package://galileo_huron_description/meshes/r_hip_pitch_link.STL" scale="1 1 1" />
         </geometry>
         <material name="grey"/>
@@ -138,5 +138,5 @@
         <origin xyz="0 0 0" rpy="0 0 0" />
         <geometry>
-            <mesh filename="package://huron_description/meshes/r_knee_pitch_link.STL" scale="1 1 1" />
+            <mesh filename="package://galileo_huron_description/meshes/r_knee_pitch_link.STL" scale="1 1 1" />
         </geometry>
         <material name="grey"/>
@@ -146,5 +146,5 @@
         <origin xyz="0 0 0" rpy="0 0 0" />
         <geometry>
-            <mesh filename="package://huron_description/meshes/r_ankle_pitch_link.STL" scale="1 1 1" />
+            <mesh filename="package://galileo_huron_description/meshes/r_ankle_pitch_link.STL" scale="1 1 1" />
         </geometry>
         <material name="">
@@ -156,5 +156,5 @@
         <origin xyz="0 0 0" rpy="0 0 0" />
         <geometry>
-            <mesh filename="package://huron_description/meshes/r_ankle_roll_link.STL" scale="1 1 1" />
+            <mesh filename="package://galileo_huron_description/meshes/r_ankle_roll_link.STL" scale="1 1 1" />
         </geometry>
         <material name="">
@@ -167,5 +167,5 @@
         <origin xyz="0 0 0" rpy=" 0 0 0" />
         <geometry>
-            <mesh filename="package://huron_description/meshes/r1_foot_ft_link.STL" scale="1 1 1" />
+            <mesh filename="package://galileo_huron_description/meshes/r1_foot_ft_link.STL" scale="1 1 1" />
         </geometry>
         <material name="green"/>
@@ -175,5 +175,5 @@
         <origin xyz="0 0 0" rpy=" 0 0 0" />
         <geometry>
-            <mesh filename="package://huron_description/meshes/r2_foot_ft_link.STL" scale="1 1 1" />
+            <mesh filename="package://galileo_huron_description/meshes/r2_foot_ft_link.STL" scale="1 1 1" />
         </geometry>
         <material name="green"/>
@@ -183,5 +183,5 @@
         <origin xyz="0 0 0" rpy=" 0 0 0" />
         <geometry>
-            <mesh filename="package://huron_description/meshes/r3_foot_ft_link.STL" scale="1 1 1" />
+            <mesh filename="package://galileo_huron_description/meshes/r3_foot_ft_link.STL" scale="1 1 1" />
         </geometry>
         <material name="green"/>
@@ -191,5 +191,5 @@
         <origin xyz="0 0 0" rpy=" 0 0 0" />
         <geometry>
-            <mesh filename="package://huron_description/meshes/r4_foot_ft_link.STL" scale="1 1 1" />
+            <mesh filename="package://galileo_huron_description/meshes/r4_foot_ft_link.STL" scale="1 1 1" />
         </geometry>
         <material name="green"/>
