Commit message: Atlas walks

File: resources/atlas/urdf/atlas.urdf (robot description, URDF)
Before this commit: robot atlas, 60 links, 59 joints
Links:
- link head: geometry visual mesh filename=package://galileo_atlas_description/meshes/head.obj
- link hokuyo_link: geometry visual mesh filename=package://galileo_atlas_description/meshes/head_camera.obj
- link l_clav: geometry visual mesh filename=package://galileo_atlas_description/meshes/r_clav.obj
- link l_foot: geometry collision sphere radius=0.0; collision sphere radius=0.0
- link l_larm: geometry visual mesh filename=package://galileo_atlas_description/meshes/r_larm.obj
- link l_lfarm: geometry visual mesh filename=package://galileo_atlas_description/meshes/r_hand.obj
- link l_lglut: geometry visual mesh filename=package://galileo_atlas_description/meshes/l_lglut.obj
- link l_lleg: geometry visual mesh filename=package://galileo_atlas_description/meshes/l_lleg.obj
- link l_scap: geometry visual mesh filename=package://galileo_atlas_description/meshes/r_scap.obj
- link l_talus: geometry visual mesh filename=package://galileo_atlas_description/meshes/l_talus.obj
- link l_uarm: geometry visual mesh filename=package://galileo_atlas_description/meshes/r_uarm.obj
- link l_ufarm: geometry visual mesh filename=package://galileo_atlas_description/meshes/r_farm.obj
- link l_uglut: geometry visual mesh filename=package://galileo_atlas_description/meshes/l_uglut.obj
- link l_uleg: geometry visual mesh filename=package://galileo_atlas_description/meshes/l_uleg.obj
- link ltorso: geometry visual mesh filename=package://galileo_atlas_description/meshes/ltorso.obj
- link mtorso: geometry visual mesh filename=package://galileo_atlas_description/meshes/mtorso.obj
- link pelvis: geometry visual mesh filename=package://galileo_atlas_description/meshes/pelvis.obj
- link r_clav: geometry visual mesh filename=package://galileo_atlas_description/meshes/r_clav.obj
- link r_foot: geometry collision sphere radius=0.0; collision sphere radius=0.0
- link r_larm: geometry visual mesh filename=package://galileo_atlas_description/meshes/r_larm.obj
- link r_lfarm: geometry visual mesh filename=package://galileo_atlas_description/meshes/r_hand.obj
- link r_lglut: geometry visual mesh filename=package://galileo_atlas_description/meshes/r_lglut.obj
- link r_lleg: geometry visual mesh filename=package://galileo_atlas_description/meshes/r_lleg.obj
- link r_scap: geometry visual mesh filename=package://galileo_atlas_description/meshes/r_scap.obj
- link r_talus: geometry visual mesh filename=package://galileo_atlas_description/meshes/r_talus.obj
- link r_uarm: geometry visual mesh filename=package://galileo_atlas_description/meshes/r_uarm.obj
- link r_ufarm: geometry visual mesh filename=package://galileo_atlas_description/meshes/r_farm.obj
- link r_uglut: geometry visual mesh filename=package://galileo_atlas_description/meshes/r_uglut.obj
- link r_uleg: geometry visual mesh filename=package://galileo_atlas_description/meshes/r_uleg.obj
- link utorso: geometry visual mesh filename=package://galileo_atlas_description/meshes/utorso.obj
