Commit message: Adding arm parameters (biqu)

File: resources/biqu_go1/biqu_go1.urdf (robot description, URDF)
Before this commit: robot robot, 23 links, 22 joints
Joints:
- joint base_to_link1: type fixed -> revolute
- joint j2: type fixed -> revolute
- joint j3: type fixed -> revolute
- joint j4: type fixed -> revolute
