Commit message: Better handling of non end-effector associated joint weights

File: resources/biqu/biqu.urdf (robot description, URDF)
Before this commit: robot robot, 23 links, 22 joints
Joints:
- joint base_to_link1: limit effort=1 velocity=20 -> lower=-3.1415 upper=3.1415 effort=1 velocity=20
- joint j2: limit effort=1 velocity=20 -> lower=-3.1415 upper=3.1415 effort=1 velocity=20
- joint j3: limit effort=1 velocity=20 -> lower=-3.1415 upper=3.1415 effort=1 velocity=20
- joint j4: limit effort=1 velocity=20 -> lower=-3.1415 upper=3.1415 effort=1 velocity=20
